File: TTLtoCANforTOF.kicad_sch (KiCad schematic)
At the start: 55 parts, among them J2 CAN, J3 TOF, J4 XT30, J6 SWD, Q1 PSMN1R4-40YLD, Q2 Q_PNP, Q3 AO4485, SW1 SW_SPST, U1 TPS54202DDC, U2 ME6211C33M5, U3 STM32G0B1CBTx, U6 TCAN3413DR, Y1 X32258MSB

Commit message: change
Parts:
- removed C22: 47uF, Capacitor_SMD:C_Elec_6.3x7.7, symbol Device:C_Polarized
- removed C23: 100nF, Capacitor_SMD:C_0603_1608Metric, symbol Device:C
- removed C24, C5: 10nF, Capacitor_SMD:C_0603_1608Metric, symbol Device:C
- removed D1: SMBJ30CA, Diode_SMD:D_SMB, symbol Device:D_TVS
- removed D3: BZX584C9V1, Diode_SMD:D_SOD-523, symbol Device:D_Schottky
- removed D4: 28-32V, Diode_SMD:D_SOD-523, symbol Device:D_Schottky
- removed Q1: PSMN1R4-40YLD, Package_TO_SOT_SMD:LFPAK56, symbol Transistor_FET:PSMN5R2-60YL
- removed Q2: Q_PNP, Package_TO_SOT_SMD:SOT-23, symbol Device:Q_PNP
- removed Q3: AO4485, Package_SO:SOP-8_3.76x4.96mm_P1.27mm, symbol Device:Q_PMOS
- removed R10, R9: 100K, Resistor_SMD:R_0603_1608Metric, symbol Device:R
- removed R11, R13: 1K, Resistor_SMD:R_0603_1608Metric, symbol Device:R
- removed R12: 10K, Resistor_SMD:R_0603_1608Metric, symbol Device:R
- removed R14, R8: 33R, Resistor_SMD:R_0603_1608Metric, symbol Device:R
- added D3: BZT52-C12, Diode_SMD:D_SOD-123, symbol Device:D_Zener
- added Q2: Si2309CDS-T1-GE3, Package_TO_SOT_SMD:SOT-23, symbol Transistor_FET:Q_PMOS_GSD
- added R8: 10kΩ, Resistor_SMD:R_0603_1608Metric, symbol Device:R_Small
- added R9: 100kΩ, Resistor_SMD:R_0603_1608Metric, symbol Device:R_Small
Connections:
- net +24V: now also D3.1 (K), Q2.3 (D), R9.2
- net GND: now also R8.1
- net VCC_IN: now also Q2.2 (S)
- new net: D3.2 (A), Q2.1 (G), R8.2, R9.1
Other:
- moved on the sheet: J2

Commit message: 1
Parts:
- removed SW1: SW_SPST, Button_Switch_SMD:SW_SPST_B3U-1000P, symbol Switch:SW_SPST
- added D1, D2: LED, LED_SMD:LED_0603_1608Metric, symbol Device:LED
- added R10, R11: 1kΩ, Resistor_SMD:R_0603_1608Metric, symbol Device:R_Small
- added TP1: RST, TestPoint:TestPoint_Pad_D1.0mm, symbol Connector:TestPoint
- added TP2: GND, TestPoint:TestPoint_Pad_D1.0mm, symbol Connector:TestPoint
- J2: footprint Connector_JST:JST_GH_SM02B-GHS-TB_1x02-1MP_P1.25mm_Horizontal -> Connector_JST:JST_GH_BM02B-GHS-TBT_1x02-1MP_P1.25mm_Vertical
- J3: footprint Connector_JST:JST_GH_SM04B-GHS-TB_1x04-1MP_P1.25mm_Horizontal -> Connector_JST:JST_GH_BM04B-GHS-TBT_1x04-1MP_P1.25mm_Vertical
Connections:
- net +24V: now also Q2.2 (S), R9.1; no longer Q2.3 (D), R9.2
- net +3.3V: now also D1.2 (A), D2.2 (A)
- net CAN+: now also J2.1 (Pin_1); no longer J2.2 (Pin_2)
- net CAN-: now also J2.2 (Pin_2); no longer J2.1 (Pin_1)
- net GND: now also R10.2, TP2.1
- net NRST: now also TP1.1
- net VCC_IN: now also Q2.3 (D); no longer Q2.2 (S)
- net at D3.2 (A), Q2.1 (G), R8.2: now also R9.2; no longer R9.1
- net LED: now reaches U3.38 (PD0)
- net LED: now also R11.2
- new net: D2.1 (K), R11.1
- new net: D1.1 (K), R10.1
- no-connect marks 35 -> 34
Other:
- moved on the sheet: D3, J2, Q2, R8, R9

Commit message: 1
Parts:
- L1: footprint Inductor_SMD:L_7.3x7.3_H3.5 -> Inductor_SMD:L_APV_ANR5020
Other:
- moved on the sheet: D3, L1, Q2, R8, R9

Commit message: fixbug
Parts:
- removed C4: 22uF, Capacitor_SMD:C_1210_3225Metric, symbol Device:C_Small
- removed C7: 75pF, Capacitor_SMD:C_0603_1608Metric, symbol Device:C_Small
- removed C8: 22uF, Capacitor_SMD:C_0805_2012Metric, symbol Device:C_Small
- removed R2: 100kΩ, Resistor_SMD:R_0603_1608Metric, symbol Device:R_Small
- removed R3: 0Ω, Resistor_SMD:R_0805_2012Metric, symbol Device:R_Small
- removed U1: TPS54202DDC, Package_TO_SOT_SMD:SOT-23-6, symbol Regulator_Switching:TPS54202DDC
- added U4: TD1469, Package_TO_SOT_SMD:SOT-23-6, symbol New_Library:TD1469
- L1: value 15uH -> 22uH
- R1: value 500kΩ -> 1MΩ
- R4: value 100kΩ -> 43kΩ
- R5: value 13.3kΩ -> 8.2kΩ
Connections:
- net +24V: now also U4.5 (VIN)
- net 5V: now also R4.1
- net GND: now also U4.2 (GND)
- net at R4.2, R5.1: now also U4.3 (FB)
- net at R1.2: now also U4.4 (EN)
- net at C1.1: now also U4.1 (BS)
- net at C1.2, L1.2: now also U4.6 (SW)
Other:
- moved on the sheet: C1, C3, C6, L1, R1, R4
