File: TTLtoCANforTOF.kicad_pcb (KiCad board)
At the start: 2 copper layers, 36 x 20.1 mm, 43 parts, among them J2 CAN, J3 TOF, J4 XT30, J6 SWD, Q2 Si2309CDS-T1-GE3, SW1 SW_SPST, U1 TPS54202DDC, U2 ME6211C33M5, U3 STM32G0B1CBTx, U6 TCAN3413DR, Y1 X32258MSB

Commit message: 1
Parts:
- removed C22: 47uF, Capacitor_SMD:C_Elec_6.3x7.7
- removed SW1: SW_SPST, Button_Switch_SMD:SW_SPST_B3U-1000P
- added D1: LED, LED_SMD:LED_0603_1608Metric, B.Cu at (153.0, 71.2)
- added D2: LED, LED_SMD:LED_0603_1608Metric, B.Cu at (166.1, 71.8)
- added R10: 1kΩ, Resistor_SMD:R_0603_1608Metric, B.Cu at (153.0, 74.3)
- added R11: 1kΩ, Resistor_SMD:R_0603_1608Metric, B.Cu at (164.4, 71.8)
- added TP1: RST, TestPoint:TestPoint_Pad_D1.0mm, B.Cu at (179.6, 62.8)
- added TP2: GND, TestPoint:TestPoint_Pad_D1.0mm, B.Cu at (181.4, 61.6)
- J2: footprint Connector_JST:JST_GH_SM02B-GHS-TB_1x02-1MP_P1.25mm_Horizontal -> Connector_JST:JST_GH_BM02B-GHS-TBT_1x02-1MP_P1.25mm_Vertical
- J3: footprint Connector_JST:JST_GH_SM04B-GHS-TB_1x04-1MP_P1.25mm_Horizontal -> Connector_JST:JST_GH_BM04B-GHS-TBT_1x04-1MP_P1.25mm_Vertical; moved to F.Cu
- J4: moved to B.Cu
- moved C11 11.1 mm to (154.4, 68.5), turned to 180 degrees
- moved C10 8.70 mm to (165.3, 68.2), turned to -90 degrees
- moved J3 8.60 mm to (154.0, 72.0), turned to 90 degrees
- moved J4 8.08 mm to (180.8, 68.9), turned to -90 degrees
- moved Q2 8.07 mm to (176.1, 74.3), turned to -90 degrees
- moved C3 7.94 mm to (172.7, 74.6)
- moved C9 6.79 mm to (163.3, 68.6), turned to -90 degrees
- moved C12 6.66 mm to (157.2, 67.0), turned to 90 degrees
- moved J6 6.38 mm to (158.6, 74.2), turned to 180 degrees
- moved L1 5.68 mm to (163.4, 72.3)
- moved C20 5.65 mm to (159.5, 67.1)
- moved C8 5.53 mm to (159.2, 65.2)
- moved R3 5.32 mm to (162.1, 62.4), turned to 90 degrees
- moved C15 5.13 mm to (173.4, 66.0), turned to 0 degrees
- moved C6 4.99 mm to (159.3, 63.1)
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Connections:
- J2 pad 1: /CAN- -> /CAN+
- J2 pad 2: /CAN+ -> /CAN-
- U3 pad 38: unconnected-(U3-PD0-Pad38) -> /LED
Routing:
- net +3.3V: track 60.8 -> 70.3 mm
- net /SWDIO: track 21.0 -> 12.3 mm
- net /USART1_TX: track 12.7 -> 17.8 mm, vias 0 -> 1
- net /NRST: track 9.52 -> 14.0 mm
- net /SWCLK: track 17.2 -> 12.8 mm
- net /LED: track 0.00 -> 4.21 mm
- net /USART1_RX: track 14.5 -> 18.3 mm, vias 0 -> 1
- net Net-(D2-K): track 0.00 -> 2.29 mm
- net Net-(D1-K): track 0.00 -> 1.57 mm
- net Net-(U1-FB): track 6.99 -> 5.56 mm
- net /CAN+: track 5.66 -> 4.32 mm
- net /CAN-: track 5.66 -> 4.32 mm
- net Net-(U1-EN): track 7.01 -> 5.71 mm
- net Net-(U1-SW): track 8.37 -> 9.25 mm
- net Net-(C7-Pad1): track 4.41 -> 3.58 mm
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Other:
- board size 36 x 20.1 mm -> 33.5 x 17.1 mm

Commit message: 1
Parts:
- L1: footprint Inductor_SMD:L_7.3x7.3_H3.5 -> Inductor_SMD:L_APV_ANR5020
- moved L1 11.4 mm to (153.9, 66.0)
- moved C20 10.2 mm to (153.5, 75.3)
- moved C6 10.1 mm to (153.3, 71.3)
- moved C8 10.1 mm to (153.3, 73.4)
- moved C3 7.80 mm to (166.4, 70.0)
- moved J3 6.20 mm to (160.2, 71.5)
- moved C4 3.32 mm to (169.9, 71.4)
- moved C7 2.60 mm to (167.2, 62.2), turned to -90 degrees
- moved U1 2.50 mm to (163.0, 64.5)
- moved R2 2.48 mm to (167.5, 65.7), turned to 90 degrees
- moved R3 2.47 mm to (159.7, 61.9), turned to 0 degrees
- moved C1 2.14 mm to (160.5, 64.5)
- moved R1 2.01 mm to (165.7, 65.6)
- moved R4 1.13 mm to (165.6, 62.2), turned to -90 degrees
- moved R5 0.93 mm to (168.7, 62.2), turned to -90 degrees
Routing:
- net 5V: track 24.8 -> 36.7 mm, vias 2 -> 1
- net /USART1_RX: track 18.3 -> 10.4 mm
- net /USART1_TX: track 17.8 -> 11.4 mm
- net Net-(C7-Pad1): track 3.58 -> 7.09 mm
- net Net-(U1-EN): track 5.71 -> 6.34 mm

Commit message: 1
Parts:
- moved C4 11.4 mm to (158.7, 69.3)
- moved J3 7.06 mm to (167.2, 71.1)
- moved C3 4.37 mm to (162.1, 69.3)
- moved C13 2.84 mm to (168.4, 63.9), turned to 90 degrees
- moved R1 2.77 mm to (162.9, 65.3)
- moved C7 2.64 mm to (164.5, 62.3)
- moved R3 2.64 mm to (157.1, 61.9)
- moved R4 2.64 mm to (162.9, 62.3)
- moved R5 2.64 mm to (166.1, 62.3)
- moved U1 2.64 mm to (160.4, 64.6)
- moved C1 2.64 mm to (157.8, 64.5)
- moved R2 2.47 mm to (165.3, 64.6), turned to 0 degrees
- moved C14 2.35 mm to (171.4, 65.6), turned to 90 degrees
- moved C20 2.01 mm to (154.8, 73.9)
- moved C6 2.01 mm to (154.6, 69.8)
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Routing:
- net +24V: track 0.00 -> 15.9 mm
- net /USART1_TX: track 11.4 -> 3.84 mm
- net 5V: track 36.7 -> 40.5 mm
- net Net-(U1-SW): track 9.19 -> 6.10 mm
- net /USART1_RX: track 10.4 -> 7.75 mm
- net GND: track 27.2 -> 29.7 mm, vias 33 -> 34
- net Net-(U1-EN): track 6.34 -> 5.48 mm
- net +3.3V: track 70.5 -> 70.3 mm, vias 3 -> 2

Commit message: fixbug
Parts:
- removed C4: 22uF, Capacitor_SMD:C_1210_3225Metric
- removed C7: 75pF, Capacitor_SMD:C_0603_1608Metric
- removed C8: 22uF, Capacitor_SMD:C_0805_2012Metric
- removed R2: 100kΩ, Resistor_SMD:R_0603_1608Metric
- removed R3: 0Ω, Resistor_SMD:R_0805_2012Metric
- removed U1: TPS54202DDC, Package_TO_SOT_SMD:SOT-23-6
- added G***: LOGO, LOGO, F.Cu at (174.5, 63.1)
- added G***: LOGO, LOGO, F.Cu at (159.5, 75.1)
- added U4: TD1469, Package_TO_SOT_SMD:SOT-23-6, F.Cu at (161.3, 66.9)
- L1: value 15uH -> 22uH
- R1: value 500kΩ -> 1MΩ
- R4: value 100kΩ -> 43kΩ
- R5: value 13.3kΩ -> 8.2kΩ
- moved C2 14.8 mm to (159.4, 63.8), turned to 0 degrees
- moved R5 9.45 mm to (161.5, 70.5), turned to 0 degrees
- moved R4 8.43 mm to (158.8, 69.6)
- moved C3 7.07 mm to (165.8, 63.3), turned to -90 degrees
- moved C6 3.01 mm to (154.9, 72.8), turned to 90 degrees
- moved R1 2.51 mm to (161.8, 63.0)
- moved C20 2.24 mm to (156.8, 72.7), turned to 90 degrees
- moved C1 2.16 mm to (158.8, 66.5), turned to 90 degrees
- moved L1 1.91 mm to (155.1, 67.5), turned to 90 degrees
Connections:
- R4 pad 1: Net-(C7-Pad1) -> 5V
Routing:
- net 5V: track 40.5 -> 32.7 mm
- net Net-(C7-Pad1): track 7.09 -> 0.00 mm
- net +24V: track 15.9 -> 19.4 mm
- net GND: track 29.7 -> 27.4 mm, vias 34 -> 56
- net Net-(U4-EN): track 5.48 -> 3.73 mm, vias 0 -> 2
- net +3.3V: track 70.3 -> 71.0 mm
- net Net-(U4-FB): track 5.60 -> 5.04 mm
- net Net-(U4-SW): track 6.10 -> 5.54 mm
Other:
- board text added: "2026.10.5"
- board text added: "Lynn"
- board text added: "TTLtoCANforTOF"

Commit message: fixbug
Parts:
- moved R1 2.50 mm to (163.7, 64.7), turned to -90 degrees
- moved C18 1.12 mm to (182.0, 63.4), turned to 0 degrees
- moved R6 0.49 mm to (180.1, 65.0)
- moved C14 0.45 mm to (171.4, 65.2)
- moved C3 0.22 mm to (166.1, 63.4)
- moved TP1 0.21 mm to (179.4, 62.8)
- moved U4 0.19 mm to (161.1, 66.9)
- moved C1 0.13 mm to (158.6, 66.5)
- moved TP2 0.06 mm to (181.3, 61.6)
Routing:
- net +3.3V: track 71.0 -> 68.5 mm
- net /USART1_RX: track 7.75 -> 5.76 mm
- net Net-(U4-EN): track 3.73 -> 1.99 mm, vias 2 -> 0
- net /NRST: track 14.0 -> 12.3 mm
- net GND: track 27.4 -> 28.5 mm
- net /USART1_TX: track 3.84 -> 4.49 mm
